File: mini/mini_rev1/aquarius-plus.kicad_sch (KiCad schematic)
At the start: 114 parts, among them J1 Power in, J2 ESP USB Host, J3 Audio out, J4 VGA, J5 ESP32 spare, J6 TF-03A, J7 FPGA spare, Q1 2N7002, SW1 SW_DPDT_x2, U1 IP4234CZ6, U2 ESP32-S3-WROOM-1-N4R2, U3 LD1117S12, U4 XC6SLX9-2TQG144C, U5 IS61C5128AL-10TLI, U6 LDL1117S33R, X1 SX3M14.31818M20F30TNN

Commit message: Generating files for first Mini PCB release
Other:
- title: Aquarius+ mini vZ80 -> Aquarius+ Mini vZ
Changed lines of the file:
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@@
 	(paper "A3")
 	(title_block
-		(title "Aquarius+ mini vZ80")
-		(date "2024-08-30")
+		(title "Aquarius+ Mini vZ")
+		(date "2024-11-27")
 		(rev "1")
 		(company "Designed by Frank van den Hoef")
